File: D16.kicad_pcb (KiCad board)
At the start: 6 copper layers, 17 x 10.9 mm, 45 parts, among them IC1 DRV8231ADSGR, IC2 NCP730BM, J1 Conn_01x08, J2 Conn_01x08, Q1 BC857BDW1, Q2 BC847BDW1, Q3 CSD87502Q2, U1 AVR-64DA32, U4 TPS22810DRVR

Commit message: Initial commit
Other:
- rule pad_to_mask_clearance: 0.2 -> 0.05
- rule solder_mask_min_width: 0.25 -> 0.1
Changed lines of the file:
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@@
     (37 F.SilkS user)
     (38 B.Mask user hide)
-    (39 F.Mask user hide)
+    (39 F.Mask user)
     (40 Dwgs.User user hide)
     (41 Cmts.User user hide)
@@
   )
   (setup
-    (last_trace_width 0.09)
+    (last_trace_width 0.15)
     (user_trace_width 0.09)
     (user_trace_width 0.15)
@@
     (pad_size 1 1)
     (pad_drill 0)
-    (pad_to_mask_clearance 0.2)
-    (solder_mask_min_width 0.25)
+    (pad_to_mask_clearance 0.05)
+    (solder_mask_min_width 0.1)
     (aux_axis_origin 0 0)
     (visible_elements 7EFFFFFF)

Commit message: Changed H-Bridge, added hardware PWM
Parts:
- removed C5: 1u/35V, Capacitor_SMD:C_0402_1005Metric
- removed U4: TPS22810DRVR, Package_DFN_QFN:DFN-6-1EP_2x2mm_P0.65mm_EP1x1.6mm
- C1, C13: value 1u -> 22u
- C2: value 100nF -> 100u/4V; footprint Capacitor_SMD:C_0402_1005Metric -> Capacitor_SMD:C_0805_2012Metric
- C4: value 2.2u/35V -> 1u/35V
- C6: value 1u/6V -> 1u
- D3: footprint _Samac:BF998215 -> RTB:BF998215
- IC1: footprint _Samac:SON50P200X200X80-9N -> RTB:SON50P200X200X80-9N
- J1: value Conn_01x08 -> Service IF
- J2: value Conn_01x08 -> NEM651
- Q3: value CSD87502Q2 -> SSM6N55NU; footprint _Samac:CSD87502Q2 -> RTB:CSD87502Q2
- R10, R12: value 68k -> 47k
- R22, R9: value 2 -> 2.2
- moved C2 3.98 mm to (61.3, -43.9), turned to 270 degrees
Connections:
- C2 pad 1: Net-(C2-Pad1) -> +3V3
- D3 pad 4: Net-(C5-Pad1) -> VHBR
- IC2 pad 7: GND -> Net-(IC2-Pad7)
Routing:
- net Net-(C5-Pad1): track 6.94 -> 0.00 mm, vias 2 -> 0
- net GND: track 29.0 -> 23.8 mm, vias 14 -> 15
- net VHBR: track 12.4 -> 15.5 mm
- net Net-(C2-Pad1): track 2.36 -> 0.00 mm
- net +3V3: vias 4 -> 5
Other:
- rule pad_to_mask_clearance: 0.05 -> 0

Commit message: mod: documentation
Parts:
- C1, C13: value 22u -> 22u/4V
- C3: value 22u/6V -> 22u/4V
- IC2: value NCP730BM -> NCP730BMT330TBG
- R10, R12: value 47k -> 33k
- R21: value 220k -> 1k
- R5: value 3.3k -> 2.2k
Connections:
- net LED.F.red renamed LED.hbt
- net LED.F.wht renamed AUX3
- net LED.R.red renamed AUX2
- net LED.R.wht renamed AUX1
- IC2 pad 7: Net-(IC2-Pad7) -> GND
Routing:
- net ISENS: track 20.3 -> 20.8 mm
Other:
- rule via_min_drill: 0.2 -> 0.3
- rule via_min_size: 0.35 -> 0.4
